Commit message: Change something

File: robot_ws/src/my_robot/src/urdf/ackerman.urdf (robot description, URDF)
Before this commit: robot em_3905, 2 links, 1 joints
Links:
- added link Laser_link; collision box size=0.05 0.05 0.05; visual box size=0.05 0.05 0.05
Joints:
- added joint laser_joint: type fixed, parent chassis, child Laser_link, origin xyz=0.1 0 0.05  rpy=0 0 0, axis 0 1 0

File: robot_ws/src/my_robot/src/urdf/ackerman_convert.urdf (robot description, URDF)
Before this commit: robot em_3905, 12 links, 11 joints
Links:
- added link Laser_link; collision boz size=0.1 0.1 0.1; visual box size=0.1 0.1 0.1
Joints:
- added joint laser_joint: type fixed, parent chassis, child Laser_link, origin xyz=0 0 0.2 rpy=0 0 0, axis 0 1 0

Commit message: Add something new

File: robot_ws/src/my_robot/src/urdf/ackerman.urdf (robot description, URDF)
Before this commit: robot em_3905, 3 links, 2 joints
Joints:
- joint laser_joint: origin xyz=0.1 0 0.05  rpy=0 0 0 -> xyz=0.1 0 0.1  rpy=0 0 0

Commit message: Update

File: robot_ws/src/my_robot/src/urdf/ackerman.urdf (robot description, URDF)
Before this commit: robot em_3905, 3 links, 2 joints
Links:
- added link Camera_link; collision box size=0.05 0.05 0.05; visual box size=0.05 0.05 0.05
Joints:
- added joint joint_camera: type fixed, parent Laser_link, child Camera_link, origin xyz=0 0 0.2  rpy=0 0 0, axis 0 1 0

Commit message: Update - code

File: robot_ws/src/my_robot/src/urdf/ackerman.urdf (robot description, URDF)
Before this commit: robot em_3905, 4 links, 3 joints
Links:
- removed link Camera_link
Joints:
- removed joint joint_camera

File: robot_ws/src/my_robot/src/urdf/ackerman_convert.urdf (robot description, URDF)
Before this commit: robot em_3905, 13 links, 12 joints
Joints:
- joint base_link_to_chassis: axis (none) -> 0 0 1; origin (none) -> xyz=0 0 0.1 rpy=0 0 0
